Commit message: fix pionner3at.urdf.xacro

File: description/urdf/pioneer3at.urdf.xacro (robot description, xacro)
@@ -197,8 +197,5 @@
 		<material value="Gazebo/Black"/>
 	</gazebo>
-	<joint name="p3at_front_${side}_wheel_joint" type="continuous">
-  	<axis xyz="0 1 0"/>
-    <anchor xyz="0 0 0"/>
-    <limit effort="100" velocity="100" />
+	<joint name="p3at_front_${side}_wheel_joint" type="fixed">
     <joint_properties damping="0.7"/>
 		<origin xyz="0 0 0" rpy="0 0 0"/>
@@ -293,8 +290,5 @@
 		<material value="Gazebo/Black"/>
 	</gazebo>
-	<joint name="p3at_back_${side}_wheel_joint" type="continuous">
-	  <axis xyz="0 1 0"/>
-    <anchor xyz="0 0 0"/>
-    <limit effort="100" velocity="100" />
+	<joint name="p3at_back_${side}_wheel_joint" type="fixed">
     <joint_properties damping="0.7"/>
 		<origin xyz="0 0 0" rpy="0 0 0"/>
